File: KicadJE_Util_RevA/KicadJE_Timeshift_Mini.sch (KiCad schematic (older format))
At the start: 48 parts

Commit message: Timeshift stage 1
Parts:
- removed C? (x2): 1u, Capacitor_SMD:C_0805_2012Metric_Pad1.15x1.40mm_HandSolder, symbol Device:C
- removed R? (x4): 20k, Resistor_SMD:R_0805_2012Metric_Pad1.15x1.40mm_HandSolder, symbol Device:R
- removed R?: 680R, Resistor_SMD:R_0805_2012Metric_Pad1.15x1.40mm_HandSolder, symbol Device:R
- removed R?: OPEN, OptoDevice:R_LDR_10x8.5mm_P7.6mm_Vertical, symbol Sensor_Optical:LDR03
- removed R?: LDR03_In2, OptoDevice:R_LDR_10x8.5mm_P7.6mm_Vertical, symbol Sensor_Optical:LDR03
- removed TP?: Flow2, TestPoint:TestPoint_THTPad_2.0x2.0mm_Drill1.0mm, symbol Connector:TestPoint
- added C? (x2): 1u, Capacitor_SMD:C_0805_2012Metric_Pad1.15x1.40mm_HandSolder, symbol Device:C
- added D? (x3): 1N4148, Diode_SMD:D_MiniMELF, symbol Device:D
- added R?: 100k, Resistor_SMD:R_0805_2012Metric_Pad1.15x1.40mm_HandSolder, symbol Device:R
- added R? (x2): 220R, Resistor_SMD:R_0805_2012Metric_Pad1.15x1.40mm_HandSolder, symbol Device:R
- added R?: OPEN, Resistor_SMD:R_0805_2012Metric_Pad1.15x1.40mm_HandSolder, symbol Device:R
- added R? (x2): 20k, Resistor_SMD:R_0805_2012Metric_Pad1.15x1.40mm_HandSolder, symbol Device:R
- added U? (x2): TL072, AJ-Dropbox-Kicad:AJ_SO-8_5.3x6.2mm_P1.27mm, symbol Amplifier_Operational:TL072
- J?: value Out1 -> Out3.1
- J?: value Out2 -> Out3.2
- J?: value In2.1 -> In3.1
- R?: value 10k -> 47k
- RV?: value 100k Glide2 -> 100k PWM1
- TP?: value Glide2 -> PWM1
Connections:
- net GND: now also C?.1, C?.1, R?.2
- net at U?.6 (-): now also RV?.2
- net at R?.2: now also R?.2, RV?.1; no longer U?.7
- net at RV?.3: now also R?.1, R?.1; no longer R?.1
- net PosPk1: now reaches R?.1
- net PosPk1: now also R?.2, U?.6 (-), U?.7; no longer RV?.1
- net In3.1a: now reaches C?.2
- net In3.1a: now also D?.1 (K), D?.1 (K), D?.2 (A), R?.1, R?.1
- net In2.1 renamed In3.1
- net In3.1: now also D?.2 (A)
- net In2.2: no longer names the net of U?.5 (+)
- net In2.2: now also R?.2
- net Out1 renamed Out3.1
- net Out3.1: now also U?.7
- net Out2 renamed Out3.2
- new net: C?.2, R?.2, U?.5 (+) (x2)
- new net: D?.1 (K), R?.1
- new net: D?.2 (A), R?.1
- new net NegPk1: R?.1, R?.2, U?.6 (-), U?.7
Other:
- moved on the sheet: C?, R?, RV?, TP?, U?B

Commit message: Update KicadJE_Timeshift_Mini.sch
Parts:
- added C?: 100n, Capacitor_SMD:C_0805_2012Metric_Pad1.15x1.40mm_HandSolder, symbol Device:C
- added R? (x4): OPEN, Resistor_SMD:R_0805_2012Metric_Pad1.15x1.40mm_HandSolder, symbol Device:R
- added R? (x2): 220R, Resistor_SMD:R_0805_2012Metric_Pad1.15x1.40mm_HandSolder, symbol Device:R
- added R? (x3): 100k, Resistor_SMD:R_0805_2012Metric_Pad1.15x1.40mm_HandSolder, symbol Device:R
- added RV?: 100k PWM2, AJ-Dropbox-Kicad:Potentiometer_China_RK09_Single_Vertical_AJ, symbol Envelope-cache-2018-08-04-13-00-04:POT
- added TP?: PWM2, AJ:Pot_6m3_scale1, symbol Connector:TestPoint
- added U?: TL072, AJ-Dropbox-Kicad:AJ_SO-8_5.3x6.2mm_P1.27mm, symbol Amplifier_Operational:TL072
Connections:
- net +12VA: now also R?.1, R?.2
- net GND: now also C?.1, R?.1, R?.2, TP?.1
- net In3.1a: now also R?.1
- net NegPk1: now also R?.1
- net Out3.1: now also R?.1
- net Out3.2: now also U?.7
- net PosPk1: now also R?.1
- net at C?.2, R?.2, U?.5 (+): now also R?.2 (x2)
- new net: C?.2, R?.2, U?.5 (+)
- new net: R?.1, R?.2, U?.6 (-)
- new net: R?.2, R?.2, RV?.1
- new net: R?.2, RV?.2
- new net: R?.1, R?.1, RV?.3
Other:
- note added: "Peak detectors"
- note added: "Slope 1 PWM"
- note added: "Slope PWM 2"
- moved on the sheet: C?, D?, R?, U?B

Commit message: annotate
Parts:
- gave numbers to parts that had none: 62

Commit message: ERC
Changed lines of the file:
@@
 Wire Wire Line
 	2400 1075 2400 1025
-Connection ~ 2525 1025
-Wire Wire Line
-	2525 1025 2600 1025
-$Comp
-L power:PWR_FLAG #FLG?
-U 1 1 5EFCD3F6
-P 2525 1025
-AR Path="/5E4B0DD9/5EFCD3F6" Ref="#FLG?"  Part="1"
-AR Path="/5E62ACA1/5EFCD3F6" Ref="#FLG?"  Part="1"
-AR Path="/5F49A670/5EFCD3F6" Ref="#FLG?"  Part="1"
-AR Path="/5EFCD3F6" Ref="#FLG?"  Part="1"
-AR Path="/5EFABE3E/5EFCD3F6" Ref="#FLG0303"  Part="1"
-F 0 "#FLG0303" H 2525 1100 50  0001 C CNN
-F 1 "PWR_FLAG" H 2675 1175 50  0000 C CNN
-F 2 "" H 2525 1025 50  0001 C CNN
-F 3 "~" H 2525 1025 50  0001 C CNN
-	1    2525 1025
-	1    0    0    -1
-$EndComp
-$Comp
-L power:PWR_FLAG #FLG?
-U 1 1 5EFCD3FC
-P 2275 1425
-AR Path="/5E4B0DD9/5EFCD3FC" Ref="#FLG?"  Part="1"
-AR Path="/5E62ACA1/5EFCD3FC" Ref="#FLG?"  Part="1"
-AR Path="/5F49A670/5EFCD3FC" Ref="#FLG?"  Part="1"
-AR Path="/5EFCD3FC" Ref="#FLG?"  Part="1"
-AR Path="/5EFABE3E/5EFCD3FC" Ref="#FLG0301"  Part="1"
-F 0 "#FLG0301" H 2275 1500 50  0001 C CNN
-F 1 "PWR_FLAG" H 2275 1598 50  0000 C CNN
-F 2 "" H 2275 1425 50  0001 C CNN
-F 3 "~" H 2275 1425 50  0001 C CNN
-	1    2275 1425
-	1    0    0    -1
-$EndComp
-$Comp
-L power:PWR_FLAG #FLG?
-U 1 1 5EFCD402
-P 2275 1825
-AR Path="/5E4B0DD9/5EFCD402" Ref="#FLG?"  Part="1"
-AR Path="/5E62ACA1/5EFCD402" Ref="#FLG?"  Part="1"
-AR Path="/5F49A670/5EFCD402" Ref="#FLG?"  Part="1"
-AR Path="/5EFCD402" Ref="#FLG?"  Part="1"
-AR Path="/5EFABE3E/5EFCD402" Ref="#FLG0302"  Part="1"
-F 0 "#FLG0302" H 2275 1900 50  0001 C CNN
-F 1 "PWR_FLAG" H 2275 1998 50  0000 C CNN
-F 2 "" H 2275 1825 50  0001 C CNN
-F 3 "~" H 2275 1825 50  0001 C CNN
-	1    2275 1825
-	1    0    0    -1
-$EndComp
 $Comp
 L Envelope-cache-2018-08-04-13-00-04:GND #PWR?
@@
 	2400 1825 2600 1825
 Connection ~ 2400 1025
-Wire Wire Line
-	2400 1025 2525 1025
 Wire Wire Line
 	2400 1425 2600 1425
@@
 Wire Notes Line
 	4500 550  4500 5325
+Wire Wire Line
+	2400 1025 2600 1025
 $EndSCHEMATC
