File: KicadJE_Util_RevA/KicadJE_Timeshift_Mini.sch (KiCad schematic (older format))
At the start: 60 parts, among them J301 In3.1, J302 Out3.1, J303 Out3.2, P301 HEADER_2x5_Doepfer, U301 TL072, U302 TL072

Commit message: Update KicadJE_Timeshift_Mini.sch
Parts:
- R312: value 100k -> OPEN
Changed lines of the file:
@@
 AR Path="/5FDBD837/5F001BCF" Ref="D?"  Part="1"
 AR Path="/5EFABE3E/5F001BCF" Ref="D304"  Part="1"
-F 0 "D304" H 2075 2600 50  0000 L CNN
-F 1 "1N1007" H 2025 2425 50  0000 L CNN
+F 0 "D304" H 2025 2425 50  0000 L CNN
+F 1 "1N1007" H 2025 2350 50  0000 L CNN
 F 2 "Diode_SMD:D_SOD-123" H 2200 2500 50  0001 C CNN
 F 3 "~" H 2200 2500 50  0001 C CNN
@@
 AR Path="/5FDBD837/5F001BFA" Ref="D?"  Part="1"
 AR Path="/5EFABE3E/5F001BFA" Ref="D305"  Part="1"
-F 0 "D305" H 2125 2675 50  0000 L CNN
+F 0 "D305" H 2100 2925 50  0000 L CNN
 F 1 "1N1007" H 2100 2850 50  0000 L CNN
 F 2 "Diode_SMD:D_SOD-123" H 2225 2775 50  0001 C CNN
@@
 AR Path="/5EFABE3E/5F32D28B" Ref="R312"  Part="1"
 F 0 "R312" V 5650 3700 50  0000 C CNN
-F 1 "100k" V 5750 3700 50  0000 C CNN
+F 1 "OPEN" V 5750 3700 50  0000 C CNN
 F 2 "Resistor_SMD:R_0805_2012Metric_Pad1.15x1.40mm_HandSolder" V 5680 3700 50  0001 C CNN
 F 3 "~" H 5750 3700 50  0001 C CNN
