File: KicadJE_Util_RevA/KicadJE_Util.kicad_pcb (KiCad board)
At the start: 2 copper layers, 159 x 128 mm, 148 parts, among them J101 RampOut1, J102 PulseOut2, J103 SawOut3, J104 In1.1, J105 In1.2, J106 In1.3, J107 SS_In2, J108 HS_In3, J109 FM_In4, J110 PWM_In5, J111 SineOut4, P101 HEADER_2x5_Doepfer, Q101 MMBT3906, Q102 UMX1N, SW101 Octave (3 state), U101 TL072, U102 TL072, U103 TL072, U104 AS3340, U105 L78L05_SOT89, U106 L79L05_SOT89, U107 TL072

Commit message: PCB Cleanup and new netlist
Parts:
- removed C107: 220p, Capacitor_SMD:C_0805_2012Metric_Pad1.15x1.40mm_HandSolder
- removed C108, C109, C114, C115, C116, C117, C118, C119: 100n, Capacitor_SMD:C_0805_2012Metric_Pad1.15x1.40mm_HandSolder
- removed C110: 1n poly, Capacitor_THT:C_Rect_L7.0mm_W2.0mm_P5.00mm
- removed C111: 1n alt, Capacitor_SMD:C_0805_2012Metric_Pad1.15x1.40mm_HandSolder
- removed C112, C113: 1u, Capacitor_SMD:C_1206_3216Metric_Pad1.42x1.75mm_HandSolder
- removed D112: 1N4148, Diode_SMD:D_SOD-123
- removed D113, D114, D117, D118: 1N1007, Diode_SMD:D_SOD-123
- removed D115: Germanium, Diode_THT:D_A-405_P7.62mm_Horizontal
- removed D116: LED, LED_SMD:LED_0805_2012Metric_Pad1.15x1.40mm_HandSolder
- removed the G*** at (70.2, 133.0)
- removed J107: SS_In2, AJ-Dropbox-Kicad:PJ301SM
- removed J108: HS_In3, AJ-Dropbox-Kicad:PJ301SM
- removed J109: FM_In4, AJ-Dropbox-Kicad:PJ301SM
- removed J110: PWM_In5, AJ-Dropbox-Kicad:PJ301SM
- removed J111: SineOut4, AJ-Dropbox-Kicad:PJ301SM
- removed JP101: Jumper, Jumper:SolderJumper-3_P1.3mm_Bridged12_Pad1.0x1.5mm_NumberLabels
- removed Q101: MMBT3906, Package_TO_SOT_SMD:SOT-23
- removed Q102: UMX1N, AJ:UMX1N_UMT6_DualNPN
- removed R132, R133, R156: 100k, Resistor_SMD:R_0805_2012Metric_Pad1.15x1.40mm_HandSolder
- removed R134, R140, R143, R158, R159, R161: 10k, Resistor_SMD:R_0805_2012Metric_Pad1.15x1.40mm_HandSolder
- removed R135, R136, R137: 47k, Resistor_SMD:R_0805_2012Metric_Pad1.15x1.40mm_HandSolder
- removed R138: 22k, Resistor_SMD:R_0805_2012Metric_Pad1.15x1.40mm_HandSolder
- removed R139, R147: 2k20, Resistor_SMD:R_0805_2012Metric_Pad1.15x1.40mm_HandSolder
- removed R141: 390R, Resistor_SMD:R_0805_2012Metric_Pad1.15x1.40mm_HandSolder
- removed R142: 18k, Resistor_SMD:R_0805_2012Metric_Pad1.15x1.40mm_HandSolder
- removed R144: 26k7, Resistor_SMD:R_0805_2012Metric_Pad1.15x1.40mm_HandSolder
- removed R145: 6k04, Resistor_SMD:R_0805_2012Metric_Pad1.15x1.40mm_HandSolder
- removed R146: 1M2, Resistor_SMD:R_0805_2012Metric_Pad1.15x1.40mm_HandSolder
- removed R148: 1k82, Resistor_SMD:R_0805_2012Metric_Pad1.15x1.40mm_HandSolder
- removed R149, R150: 13k3, Resistor_SMD:R_0805_2012Metric_Pad1.15x1.40mm_HandSolder
- removed R151, R163: OPEN, Resistor_SMD:R_0805_2012Metric_Pad1.15x1.40mm_HandSolder
- removed R152: 0R, Resistor_SMD:R_0805_2012Metric_Pad1.15x1.40mm_HandSolder
- removed R153, R155, R164: 1k, Resistor_SMD:R_0805_2012Metric_Pad1.15x1.40mm_HandSolder
- removed R154: 3k, Resistor_SMD:R_0805_2012Metric_Pad1.15x1.40mm_HandSolder
- removed R157: 15k, Resistor_SMD:R_0805_2012Metric_Pad1.15x1.40mm_HandSolder
- removed R160, R162: 25k, Resistor_SMD:R_0805_2012Metric_Pad1.15x1.40mm_HandSolder
- removed SW101: Octave (3 state), AJ-Dropbox-Kicad:SP1MS1
- removed U103, U107: TL072, AJ-Dropbox-Kicad:AJ_SO-8_5.3x6.2mm_P1.27mm
- removed U104: AS3340, Package_DIP:DIP-16_W10.16mm_LongPads
- removed U105: L78L05_SOT89, Package_TO_SOT_SMD:SOT-89-3
- removed U106: L79L05_SOT89, Package_TO_SOT_SMD:SOT-89-3
- added C201: 1u, Capacitor_SMD:C_1206_3216Metric_Pad1.42x1.75mm_HandSolder, F.Cu at (64.4, -12.6)
- added C202: 1u, Capacitor_SMD:C_1206_3216Metric_Pad1.42x1.75mm_HandSolder, F.Cu at (70.4, -11.8)
- added C203: 100n, Capacitor_SMD:C_0805_2012Metric_Pad1.15x1.40mm_HandSolder, F.Cu at (138.6, -47.1)
- added C204: 100n, Capacitor_SMD:C_0805_2012Metric_Pad1.15x1.40mm_HandSolder, F.Cu at (103.5, -13.9)
- added C205: 100n, Capacitor_SMD:C_0805_2012Metric_Pad1.15x1.40mm_HandSolder, F.Cu at (124.4, -34.7)
- added C206: 100n, Capacitor_SMD:C_0805_2012Metric_Pad1.15x1.40mm_HandSolder, F.Cu at (114.0, -22.9)
- added C207: OPEN, Capacitor_SMD:C_0805_2012Metric_Pad1.15x1.40mm_HandSolder, F.Cu at (133.2, -46.4)
- added C208: 1u, Capacitor_SMD:C_0805_2012Metric_Pad1.15x1.40mm_HandSolder, F.Cu at (108.2, -19.6)
- added C209: 1u, Capacitor_SMD:C_0805_2012Metric_Pad1.15x1.40mm_HandSolder, F.Cu at (138.6, -50.1)
- added C210: 1u, Capacitor_SMD:C_0805_2012Metric_Pad1.15x1.40mm_HandSolder, F.Cu at (103.5, -16.9)
- added C211: 4u7, Capacitor_SMD:C_0805_2012Metric_Pad1.15x1.40mm_HandSolder, F.Cu at (108.2, -16.6)
- added C212: OPEN, Capacitor_SMD:C_0805_2012Metric_Pad1.15x1.40mm_HandSolder, F.Cu at (133.2, -40.5)
- added C301: 1u, Capacitor_SMD:C_1206_3216Metric_Pad1.42x1.75mm_HandSolder, F.Cu at (91.5, 30.5)
- added C302: 1u, Capacitor_SMD:C_1206_3216Metric_Pad1.42x1.75mm_HandSolder, F.Cu at (101.7, 17.1)
- added C303: 100n, Capacitor_SMD:C_0805_2012Metric_Pad1.15x1.40mm_HandSolder, F.Cu at (122.9, 9.14)
- added C304: 100n, Capacitor_SMD:C_0805_2012Metric_Pad1.15x1.40mm_HandSolder, F.Cu at (74.6, 25.8)
- added C305: 100n, Capacitor_SMD:C_0805_2012Metric_Pad1.15x1.40mm_HandSolder, F.Cu at (59.1, 33.7)
- added C306: 100n, Capacitor_SMD:C_0805_2012Metric_Pad1.15x1.40mm_HandSolder, F.Cu at (59.1, 36.7)
- added C307: OPEN, Capacitor_SMD:C_0805_2012Metric_Pad1.15x1.40mm_HandSolder, F.Cu at (74.6, 28.8)
- added C308: 100n, Capacitor_SMD:C_0805_2012Metric_Pad1.15x1.40mm_HandSolder, F.Cu at (118.1, 10.4)
- added C309: 1u, Capacitor_SMD:C_0805_2012Metric_Pad1.15x1.40mm_HandSolder, F.Cu at (107.0, 16.9)
- added C310: 1u, Capacitor_SMD:C_0805_2012Metric_Pad1.15x1.40mm_HandSolder, F.Cu at (90.9, 33.6)
- added D111: 1N1007, Diode_SMD:D_SOD-123, F.Cu at (172.9, -17.5)
- added D201: 1N1007, Diode_SMD:D_SOD-123, F.Cu at (117.1, -30.7)
- added D202: 1N1007, Diode_SMD:D_SOD-123, F.Cu at (93.5, -12.0)
- added D203: LED, LED_SMD:LED_0805_2012Metric_Pad1.15x1.40mm_HandSolder, F.Cu at (59.1, -46.4)
- added D204: 1N1007, Diode_SMD:D_SOD-123, F.Cu at (108.8, -25.7)
- added D205: LED, LED_THT:LED_D3.0mm, F.Cu at (96.9, -18.5)
- added D206: 1N1007, Diode_SMD:D_SOD-123, F.Cu at (76.2, -11.8)
- added D207: LED, LED_THT:LED_D3.0mm, F.Cu at (132.0, -50.7)
- added D208: 1N1007, Diode_SMD:D_SOD-123, F.Cu at (82.0, -11.8)
- added D209: 1N1007, Diode_SMD:D_SOD-123, F.Cu at (87.7, -12.0)
- added D301: 1N1007, Diode_SMD:D_SOD-123, F.Cu at (105.2, 20.4)
- added D302: 1N1007, Diode_SMD:D_SOD-123, F.Cu at (99.4, 20.5)
- added D303: LED, LED_SMD:LED_0805_2012Metric_Pad1.15x1.40mm_HandSolder, F.Cu at (59.1, 11.5)
- added D304: 1N1007, Diode_SMD:D_SOD-123, F.Cu at (123.0, 0.09)
- added D305: 1N1007, Diode_SMD:D_SOD-123, F.Cu at (99.4, 23.8)
- added D306: 1N4148, Diode_SMD:D_MiniMELF, F.Cu at (108.2, 13.8)
- added D307: 1N4148, Diode_SMD:D_MiniMELF, F.Cu at (112.6, 10.5)
- added D308: 1N4148, Diode_SMD:D_MiniMELF, F.Cu at (101.9, 13.8)
- added H201: ON, AJ:LED_Hole_3mm, F.Cu at (122.8, -42.4)
- added H202: MountingHole_Pad, AJ:MountingHole_Eurorack3, F.Cu at (135.5, -62.0)
- added H203: MountingHole_Pad, AJ:MountingHole_Eurorack3, F.Cu at (110.2, -29.9)
- added H204: MountingHole_Pad, AJ:MountingHole_Eurorack3, F.Cu at (135.5, -57.0)
- added H205: MountingHole_Pad, AJ:MountingHole_Eurorack3, F.Cu at (65.5, -16.7)
- added H301: ON, AJ:LED_Hole_3mm, F.Cu at (83.5, 36.4)
- added H302: MountingHole_Pad, AJ:MountingHole_Eurorack3, F.Cu at (124.1, -4.09)
- added H303: MountingHole_Pad, AJ:MountingHole_Eurorack3, F.Cu at (92.5, 21.3)
- added H304: MountingHole_Pad, AJ:MountingHole_Eurorack3, F.Cu at (92.5, 26.3)
- added H305: MountingHole_Pad, AJ:MountingHole_Eurorack3, F.Cu at (76.2, 35.7)
- added J201: Out2.1, AJ-Dropbox-Kicad:PJ301SM, F.Cu at (103.4, -57.9)
- added J202: Out2.2, AJ-Dropbox-Kicad:PJ301SM, F.Cu at (93.3, -57.9)
- added J203: In2.1, AJ-Dropbox-Kicad:PJ301SM, F.Cu at (67.1, -41.3)
- added J204: CV2.1, AJ-Dropbox-Kicad:PJ301SM, F.Cu at (77.3, -41.3)
- added J205: In2.2, AJ-Dropbox-Kicad:PJ301SM, F.Cu at (87.4, -43.6)
- added J206: CV2.2, AJ-Dropbox-Kicad:PJ301SM, F.Cu at (67.1, -27.0)
- added J301: In3.1, AJ-Dropbox-Kicad:PJ301SM, F.Cu at (67.1, 30.9)
- added J302: Out3.1, AJ-Dropbox-Kicad:PJ301SM, F.Cu at (93.3, -0.01)
- added J303: Out3.2, AJ-Dropbox-Kicad:PJ301SM, F.Cu at (82.6, 14.3)
- added P201: HEADER_2x5_Doepfer, Connector_IDC:IDC-Header_2x05_P2.54mm_Vertical, F.Cu at (50.2, -58.3)
- added P301: HEADER_2x5_Doepfer, Connector_IDC:IDC-Header_2x05_P2.54mm_Vertical, F.Cu at (50.2, -0.43)
- added R201: 22k, Resistor_SMD:R_0805_2012Metric_Pad1.15x1.40mm_HandSolder, F.Cu at (122.4, -31.8)
- added R202: OPEN, Resistor_SMD:R_0805_2012Metric_Pad1.15x1.40mm_HandSolder, F.Cu at (133.2, -43.5)
- added R203: OPEN, Resistor_SMD:R_0805_2012Metric_Pad1.15x1.40mm_HandSolder, F.Cu at (118.8, -27.5)
- added R204: 680R, Resistor_SMD:R_0805_2012Metric_Pad1.15x1.40mm_HandSolder, F.Cu at (103.5, -19.8)
- added R205: 680R, Resistor_SMD:R_0805_2012Metric_Pad1.15x1.40mm_HandSolder, F.Cu at (128.5, -44.2)
- added R206: 10k, Resistor_SMD:R_0805_2012Metric_Pad1.15x1.40mm_HandSolder, F.Cu at (108.3, -22.5)
- added R207: 10k, Resistor_SMD:R_0805_2012Metric_Pad1.15x1.40mm_HandSolder, F.Cu at (119.7, -34.7)
- added R208: 10k, Resistor_SMD:R_0805_2012Metric_Pad1.15x1.40mm_HandSolder, F.Cu at (124.4, -37.7)
- added R209: 10k, Resistor_SMD:R_0805_2012Metric_Pad1.15x1.40mm_HandSolder, F.Cu at (118.8, -21.6)
- added R210: 10k, Resistor_SMD:R_0805_2012Metric_Pad1.15x1.40mm_HandSolder, F.Cu at (108.2, -13.7)
- added R211: 10k, Resistor_SMD:R_0805_2012Metric_Pad1.15x1.40mm_HandSolder, F.Cu at (119.7, -37.7)
- added R212: 20k, Resistor_SMD:R_0805_2012Metric_Pad1.15x1.40mm_HandSolder, F.Cu at (138.6, -53.0)
- added R213: 20k, Resistor_SMD:R_0805_2012Metric_Pad1.15x1.40mm_HandSolder, F.Cu at (98.7, -14.3)
- added R214: 20k, Resistor_SMD:R_0805_2012Metric_Pad1.15x1.40mm_HandSolder, F.Cu at (114.0, -25.9)
- added R215: 20k, Resistor_SMD:R_0805_2012Metric_Pad1.15x1.40mm_HandSolder, F.Cu at (98.7, -11.3)
- added R216: OPEN, OptoDevice:R_LDR_10x8.5mm_P7.6mm_Vertical, F.Cu at (74.4, -18.5)
- added R217: LDR03_In2, OptoDevice:R_LDR_10x8.5mm_P7.6mm_Vertical, F.Cu at (74.4, -28.5)
- added R218: 20k, Resistor_SMD:R_0805_2012Metric_Pad1.15x1.40mm_HandSolder, F.Cu at (128.5, -41.3)
- added R219: 20k, Resistor_SMD:R_0805_2012Metric_Pad1.15x1.40mm_HandSolder, F.Cu at (113.0, -19.6)
- added R220: 220R, Resistor_SMD:R_0805_2012Metric_Pad1.15x1.40mm_HandSolder, F.Cu at (113.0, -16.6)
- added R221: 220R, Resistor_SMD:R_0805_2012Metric_Pad1.15x1.40mm_HandSolder, F.Cu at (127.1, -31.8)
- added R222: 680R, Resistor_SMD:R_0805_2012Metric_Pad1.15x1.40mm_HandSolder, F.Cu at (133.9, -37.6)
- added R223: 680R, Resistor_SMD:R_0805_2012Metric_Pad1.15x1.40mm_HandSolder, F.Cu at (138.0, -41.2)
- added R224: OPEN, Resistor_SMD:R_0805_2012Metric_Pad1.15x1.40mm_HandSolder, F.Cu at (123.5, -28.8)
- added R225: OPEN, Resistor_SMD:R_0805_2012Metric_Pad1.15x1.40mm_HandSolder, F.Cu at (138.0, -44.2)
- added R226: 20k, Resistor_SMD:R_0805_2012Metric_Pad1.15x1.40mm_HandSolder, F.Cu at (129.2, -37.6)
- added R227: 20k, Resistor_SMD:R_0805_2012Metric_Pad1.15x1.40mm_HandSolder, F.Cu at (118.8, -24.6)
- added R228: LDR03_In1, OptoDevice:R_LDR_10x8.5mm_P7.6mm_Vertical, F.Cu at (110.7, -59.5)
- added R229: OPEN, OptoDevice:R_LDR_10x8.5mm_P7.6mm_Vertical, F.Cu at (94.7, -45.1)
- added R301: 22k, Resistor_SMD:R_0805_2012Metric_Pad1.15x1.40mm_HandSolder, F.Cu at (103.7, 27.0)
- added R302: 10k, Resistor_SMD:R_0805_2012Metric_Pad1.15x1.40mm_HandSolder, F.Cu at (93.9, 36.5)
- added R303: OPEN, Resistor_SMD:R_0805_2012Metric_Pad1.15x1.40mm_HandSolder, F.Cu at (122.5, 6.19)
- added R304: OPEN, Resistor_SMD:R_0805_2012Metric_Pad1.15x1.40mm_HandSolder, F.Cu at (96.9, 33.2)
- added R305: 1k, Resistor_SMD:R_0805_2012Metric_Pad1.15x1.40mm_HandSolder, F.Cu at (98.9, 27.0)
- added R306: 1k, Resistor_SMD:R_0805_2012Metric_Pad1.15x1.40mm_HandSolder, F.Cu at (122.5, 3.24)
- added R307: 47k, Resistor_SMD:R_0805_2012Metric_Pad1.15x1.40mm_HandSolder, F.Cu at (96.9, 30.3)
- added R308: OPEN, Resistor_SMD:R_0805_2012Metric_Pad1.15x1.40mm_HandSolder, F.Cu at (113.8, 13.6)
- added R309: 220R, Resistor_SMD:R_0805_2012Metric_Pad1.15x1.40mm_HandSolder, F.Cu at (110.4, 19.9)
- added R310: 100k, Resistor_SMD:R_0805_2012Metric_Pad1.15x1.40mm_HandSolder, F.Cu at (98.6, 36.2)
- added R311: 100k, Resistor_SMD:R_0805_2012Metric_Pad1.15x1.40mm_HandSolder, F.Cu at (101.6, 29.9)
- added R312: 100k, Resistor_SMD:R_0805_2012Metric_Pad1.15x1.40mm_HandSolder, F.Cu at (110.4, 22.8)
- added R313: OPEN, Resistor_SMD:R_0805_2012Metric_Pad1.15x1.40mm_HandSolder, F.Cu at (119.9, 19.2)
- added R314: 220R, Resistor_SMD:R_0805_2012Metric_Pad1.15x1.40mm_HandSolder, F.Cu at (113.8, 16.6)
- added R315: 220R, Resistor_SMD:R_0805_2012Metric_Pad1.15x1.40mm_HandSolder, F.Cu at (115.2, 22.5)
- added R316: 100k, Resistor_SMD:R_0805_2012Metric_Pad1.15x1.40mm_HandSolder, F.Cu at (123.3, 12.1)
- added R317: 220R, Resistor_SMD:R_0805_2012Metric_Pad1.15x1.40mm_HandSolder, F.Cu at (106.4, 29.9)
- added R318: OPEN, Resistor_SMD:R_0805_2012Metric_Pad1.15x1.40mm_HandSolder, F.Cu at (108.4, 26.5)
- added R319: OPEN, Resistor_SMD:R_0805_2012Metric_Pad1.15x1.40mm_HandSolder, F.Cu at (89.1, 36.5)
- added R320: 220R, Resistor_SMD:R_0805_2012Metric_Pad1.15x1.40mm_HandSolder, F.Cu at (118.5, 16.3)
- added R321: 20k, Resistor_SMD:R_0805_2012Metric_Pad1.15x1.40mm_HandSolder, F.Cu at (101.6, 32.9)
- added R322: 20k, Resistor_SMD:R_0805_2012Metric_Pad1.15x1.40mm_HandSolder, F.Cu at (115.2, 19.5)
- added R323: OPEN, Resistor_SMD:R_0805_2012Metric_Pad1.15x1.40mm_HandSolder, F.Cu at (104.7, 23.6)
- added R324: OPEN, Resistor_SMD:R_0805_2012Metric_Pad1.15x1.40mm_HandSolder, F.Cu at (118.5, 13.3)
- added RV201: 100k Glide1, AJ-Dropbox-Kicad:Potentiometer_China_RK09_Single_Vertical_AJ, F.Cu at (74.4, -54.8)
- added RV202: 100k Glide2, AJ-Dropbox-Kicad:Potentiometer_China_RK09_Single_Vertical_AJ, F.Cu at (47.7, -16.0)
- added RV301: 100k PWM1, AJ-Dropbox-Kicad:Potentiometer_China_RK09_Single_Vertical_AJ, F.Cu at (74.4, 3.09)
- added RV302: 100k PWM2, AJ-Dropbox-Kicad:Potentiometer_China_RK09_Single_Vertical_AJ, F.Cu at (63.7, 19.7)
- added TP108: OFF2, AJ:Pot_6m3_scale1, F.Cu at (154.6, -33.7)
- added TP109: Gain2, AJ:Pot_6m3_scale1, F.Cu at (165.4, -55.9)
- added TP110: Gain1, AJ:Pot_6m3_scale1, F.Cu at (181.4, -55.9)
- added TP111: Flow1, TestPoint:TestPoint_THTPad_2.0x2.0mm_Drill1.0mm, F.Cu at (209.9, -23.1)
- added TP112: Flow2, TestPoint:TestPoint_THTPad_2.0x2.0mm_Drill1.0mm, F.Cu at (204.5, -17.2)
- added TP201: Tri, AJ:Jack_6m3, F.Cu at (111.8, -37.9)
- added TP202: SQ, AJ:Jack_6m3, F.Cu at (100.7, -34.6)
- added TP203: In1, AJ:Jack_6m3, F.Cu at (89.7, -30.3)
- added TP204: In2, AJ:Jack_6m3, F.Cu at (89.7, -19.2)
- added TP205: In3, AJ:Jack_6m3, F.Cu at (126.0, -59.0)
- added TP206: SS, AJ:Jack_6m3, F.Cu at (114.0, -48.9)
- added TP207: Glide1, AJ:Pot_6m3_scale1, F.Cu at (54.0, -33.7)
- added TP208: Glide2, AJ:Pot_6m3_scale1, F.Cu at (64.7, -55.9)
- added TP209: Flow1, TestPoint:TestPoint_THTPad_2.0x2.0mm_Drill1.0mm, F.Cu at (141.5, -62.5)
- added TP210: Flow2, TestPoint:TestPoint_THTPad_2.0x2.0mm_Drill1.0mm, F.Cu at (106.5, -48.1)
- added TP301: In1, AJ:Jack_6m3, F.Cu at (93.2, 13.3)
- added TP302: Tri, AJ:Jack_6m3, F.Cu at (103.9, -1.06)
- added TP303: SQ, AJ:Jack_6m3, F.Cu at (83.0, 27.6)
- added TP304: PWM1, AJ:Pot_6m3_scale1, F.Cu at (54.0, 24.2)
- added TP305: PWM2, AJ:Pot_6m3_scale1, F.Cu at (64.7, 1.99)
- added U201: TL072, AJ-Dropbox-Kicad:AJ_SO-8_5.3x6.2mm_P1.27mm, F.Cu at (100.6, -25.2)
- added U202: TL072, AJ-Dropbox-Kicad:AJ_SO-8_5.3x6.2mm_P1.27mm, F.Cu at (124.9, -49.6)
- added U301: TL072, AJ-Dropbox-Kicad:AJ_SO-8_5.3x6.2mm_P1.27mm, F.Cu at (51.4, 36.1)
- added U302: TL072, AJ-Dropbox-Kicad:AJ_SO-8_5.3x6.2mm_P1.27mm, F.Cu at (114.8, -2.71)
- added U303: TL072, AJ-Dropbox-Kicad:AJ_SO-8_5.3x6.2mm_P1.27mm, F.Cu at (104.1, 8.34)
- added U304: TL072, AJ-Dropbox-Kicad:AJ_SO-8_5.3x6.2mm_P1.27mm, F.Cu at (114.8, 5.04)
- C101: value 100n -> 1u; footprint Capacitor_SMD:C_0805_2012Metric_Pad1.15x1.40mm_HandSolder -> Capacitor_SMD:C_1206_3216Metric_Pad1.42x1.75mm_HandSolder; moved to F.Cu
- C102: value 1n -> 1u; footprint Capacitor_SMD:C_0805_2012Metric_Pad1.15x1.40mm_HandSolder -> Capacitor_SMD:C_1206_3216Metric_Pad1.42x1.75mm_HandSolder; moved to F.Cu
- C103: value 1n -> 100n; moved to F.Cu
- C104, C105, C106: value 10n -> 100n; moved to F.Cu
- D101, D102, D104, D105, D106, D107, D108, P101, R105, U101, U102: moved to F.Cu
- D103: value 1N1007 -> LED; footprint Diode_SMD:D_SOD-123 -> LED_SMD:LED_0805_2012Metric_Pad1.15x1.40mm_HandSolder; moved to F.Cu
- J101: value RampOut1 -> Out1
- J102: value PulseOut2 -> Out2
- J103: value SawOut3 -> In1.1
- J104: value In1.1 -> In1.2
- J105: value In1.2 -> In1.3
- J106: value In1.3 -> SS_In2
- R101: value 47k -> 22k; moved to F.Cu
- R102: value 470R -> OPEN; moved to F.Cu
- R103: value 82k -> OPEN; moved to F.Cu
- R104: value 20k -> 1k; moved to F.Cu
- R106: value 910R -> 100k; moved to F.Cu
- R107, R111, R112, R113, R116: value 1k -> 10k; moved to F.Cu
- R108, R109, R110, R122, R123: value 100k -> 10k; moved to F.Cu
- R114: value 1k6 -> 10k; moved to F.Cu
- R115: value 1M -> 10k; moved to F.Cu
- R117: value 360k -> 100k; moved to F.Cu
- R118: value 470R -> 20k; moved to F.Cu
- R119: value 1M -> 20k; moved to F.Cu
- R120: value 100k -> 20k; moved to F.Cu
- R121, R128: value 12k5 -> 20k; moved to F.Cu
- R124: value 100k -> 1k; moved to F.Cu
- R125: value 470R -> 1k; moved to F.Cu
- R126, R127: value 10k -> OPEN; moved to F.Cu
- R129: value 1M5 -> 20k; moved to F.Cu
- R130, R131: value 10k -> 1k; moved to F.Cu
- RV101: value 100k Fine -> 100k Offset1
- RV102: value 100k PWM -> 100k Gain1
- RV103: value 5k -> 100k Gain2; footprint Potentiometer_THT:Potentiometer_Bourns_3296W_Vertical -> AJ-Dropbox-Kicad:Potentiometer_China_RK09_Single_Vertical_AJ; moved to F.Cu
- RV104: value 50k -> 100k Offset2; footprint Potentiometer_THT:Potentiometer_Bourns_3296W_Vertical -> AJ-Dropbox-Kicad:Potentiometer_China_RK09_Single_Vertical_AJ; moved to F.Cu
- TP107: renamed from TP113; value PWM -> OFF1
- moved C103 268.9 mm to (233.3, -57.1), turned to 0 degrees
- moved D108 266.4 mm to (228.1, -56.1)
- moved D105 259.2 mm to (228.1, -59.5)
- moved R122 258.5 mm to (233.3, -63.0), turned to 0 degrees
- moved R111 254.9 mm to (226.7, -47.1)
- moved R113 251.3 mm to (232.3, -50.0)
- moved R131 244.4 mm to (231.5, -47.1), turned to 0 degrees
- moved R107 237.1 mm to (232.3, -53.0), turned to 0 degrees
- moved D109 236.3 mm to (228.1, -62.8), turned to 0 degrees
- moved R110 236.2 mm to (227.6, -53.0)
- moved R115 234.0 mm to (226.7, -44.1), turned to 0 degrees
- moved R121 229.2 mm to (216.2, -45.3), turned to 0 degrees
- moved R118 226.8 mm to (221.0, -42.8), turned to 0 degrees
- moved C105 224.8 mm to (222.0, -45.7), turned to 0 degrees
- moved J106 221.6 mm to (210.0, -57.9), turned to 0 degrees
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- renumbered H105 to H101, H101 to H102, H102 to H103, H103 to H104, H104 to H105, TP109 to TP101, TP110 to TP102, TP102 to TP103, TP103 to TP104, TP104 to TP105, TP105 to TP106
Connections:
- C101 pad 1: Net-(C101-Pad1) -> +12VA
- C101 pad 2: Net-(C101-Pad2) -> GND
- C102 pad 1: 3SoftSyncIn2 -> GND
- C102 pad 2: Net-(C102-Pad2) -> -12VA
- C103 pad 1: 3HardSyncIn3 -> +12VA
- C103 pad 2: Net-(C103-Pad2) -> GND
- C104 pad 2: Net-(C104-Pad2) -> -12VA
- C105 pad 1: -12VA -> +12VA
- C105 pad 2: Net-(C105-Pad2) -> GND
- C106 pad 1: Net-(C106-Pad1) -> GND
- C106 pad 2: 3PWM_In5 -> -12VA
- D101 pad 2: Net-(D101-Pad2) -> GND
- D102 pad 1: Net-(D101-Pad2) -> GND
- D102 pad 2: -5V -> -12VA
- D103 pad 1: +12VA -> -12VA
- D104 pad 1: Net-(D103-Pad2) -> +12VA
- D104 pad 2: GND -> Net-(D104-Pad2)
- D105 pad 2: 3SoftSyncIn2 -> Net-(D105-Pad2)
- D106 pad 2: 3HardSyncIn3 -> Net-(D106-Pad2)
- D107 pad 1: 3SoftSyncIn2 -> +12VA
- D107 pad 2: GND -> Net-(D107-Pad2)
- D108 pad 1: 3HardSyncIn3 -> Net-(D104-Pad2)
- D108 pad 2: GND -> -12VA
- D109 pad 1: +12VA -> Net-(D105-Pad2)
- D109 pad 2: 3FM_Lin_In4 -> -12VA
- D110 pad 1: 3FM_Lin_In4 -> Net-(D106-Pad2)
- J103 pad TN: (no net) -> GND
- R101 pad 1: Net-(R101-Pad1) -> Net-(D103-Pad2)
- R101 pad 2: +5V -> GND
- R102 pad 1: Net-(R102-Pad1) -> GND
- R102 pad 2: GND -> Net-(J101-PadT)
- R103 pad 1: 3Octave -> GND
- R103 pad 2: +5V -> Net-(J102-PadT)
- R104 pad 1: Net-(R102-Pad1) -> Out1
- R104 pad 2: 3Octave -> Net-(J101-PadT)
- R105 pad 1: Net-(R105-Pad1) -> Out2
- R105 pad 2: Net-(J101-PadT) -> Net-(J102-PadT)
- R106 pad 1: GND -> Net-(R106-Pad1)
- R106 pad 2: Net-(J102-PadT) -> Out1
- R107 pad 1: Net-(R107-Pad1) -> Net-(D104-Pad2)
- R108 pad 1: Net-(D103-Pad2) -> Net-(D105-Pad2)
- R109 pad 1: Net-(D103-Pad2) -> Net-(D106-Pad2)
- R110 pad 1: Net-(D103-Pad2) -> Net-(D107-Pad2)
- R111 pad 1: Net-(C102-Pad2) -> Flow1
- R111 pad 2: Net-(J107-PadT) -> Net-(R111-Pad2)
- R112 pad 1: Net-(C103-Pad2) -> Net-(R112-Pad1)
- R112 pad 2: Net-(J108-PadT) -> Net-(R106-Pad1)
- R113 pad 1: Net-(D101-Pad2) -> In1
- R113 pad 2: Net-(J110-PadT) -> Net-(D104-Pad2)
- R114 pad 1: Net-(R107-Pad1) -> Inv1
- R114 pad 2: GND -> Net-(D105-Pad2)
- R115 pad 1: 3FM_Lin_In4 -> In2
- R115 pad 2: Net-(C101-Pad1) -> Net-(D106-Pad2)
- R116 pad 1: Net-(R116-Pad1) -> Inv2
- R116 pad 2: Net-(J102-PadT) -> Net-(D107-Pad2)
- R117 pad 1: Net-(D103-Pad2) -> Net-(R117-Pad1)
- R117 pad 2: +12VA -> Out2
- R118 pad 1: Net-(C104-Pad2) -> In1
- R118 pad 2: Net-(D103-Pad2) -> GND
- R119 pad 1: Net-(R119-Pad1) -> Inv1
- R119 pad 2: 3CVIn1 -> GND
- R120 pad 1: Net-(R120-Pad1) -> In2
- R120 pad 2: Net-(R116-Pad1) -> GND
- R121 pad 1: Net-(R121-Pad1) -> Inv2
- R121 pad 2: Net-(R107-Pad1) -> GND
- R122 pad 1: Net-(C106-Pad1) -> Flow2
- R122 pad 2: Net-(D101-Pad2) -> Net-(R122-Pad2)
- R123 pad 1: Net-(C106-Pad1) -> Net-(R123-Pad1)
- R123 pad 2: 3PWM_Adj -> Net-(R117-Pad1)
- R124 pad 1: Net-(C106-Pad1) -> Net-(R124-Pad1)
- R124 pad 2: -5V -> Inv1
- R125 pad 1: Net-(C105-Pad2) -> Net-(R125-Pad1)
- R125 pad 2: 3FM_Lin_In4 -> Inv2
- R126 pad 1: 3VP_2 -> Net-(R126-Pad1)
- R126 pad 2: Net-(R126-Pad2) -> Net-(R124-Pad1)
- R127 pad 1: 3VSO_3 -> Net-(R127-Pad1)
- R127 pad 2: Net-(R127-Pad2) -> Net-(R125-Pad1)
- R128 pad 1: -5V -> Net-(R126-Pad1)
- R128 pad 2: Net-(R127-Pad2) -> Net-(R128-Pad2)
- R129 pad 1: +12VA -> Net-(R127-Pad1)
- R129 pad 2: 3FM_Lin_In4 -> Net-(R129-Pad2)
- R130 pad 1: GND -> Flow1
- R130 pad 2: Net-(R120-Pad1) -> Net-(R128-Pad2)
- R131 pad 1: GND -> Flow2
- R131 pad 2: Net-(R121-Pad1) -> Net-(R129-Pad2)
- RV101 pad 2: Net-(R119-Pad1) -> Net-(R112-Pad1)
- RV102 pad 1: GND -> Net-(R126-Pad1)
- RV102 pad 2: Net-(R133-Pad1) -> Net-(R124-Pad1)
- RV102 pad 3: +12VA -> Inv1
- RV103 pad 1: -5V -> Net-(R127-Pad1)
- RV103 pad 2: -5V -> Net-(R125-Pad1)
- RV103 pad 3: Net-(R144-Pad2) -> Inv2
- RV104 pad 1: Net-(Q102-Pad1) -> -12VA
- RV104 pad 2: Net-(R142-Pad1) -> Net-(R123-Pad1)
- RV104 pad 3: Net-(Q102-Pad4) -> +12VA
- U101 pad 1: Net-(R116-Pad1) -> Out2
- U101 pad 2: Net-(R120-Pad1) -> Net-(R117-Pad1)
- U101 pad 3: Net-(R126-Pad2) -> Net-(R122-Pad2)
- U101 pad 5: 3VTO_1 -> Net-(R111-Pad2)
- U101 pad 6: Net-(R105-Pad1) -> Net-(R106-Pad1)
- U101 pad 7: Net-(R105-Pad1) -> Out1
- U102 pad 1: 3PWM_In5 -> Net-(R128-Pad2)
- U102 pad 2: Net-(C106-Pad1) -> Inv1
- U102 pad 3: GND -> In1
- U102 pad 5: Net-(R127-Pad2) -> In2
- U102 pad 6: Net-(R121-Pad1) -> Inv2
- U102 pad 7: Net-(R107-Pad1) -> Net-(R129-Pad2)
Routing:
- net +12VA: track 297.1 -> 0.00 mm, vias 7 -> 0
- net -12VA: track 193.5 -> 0.00 mm, vias 5 -> 0
- net -5V: track 182.7 -> 0.00 mm, vias 8 -> 0
- net GND: track 110.0 -> 0.00 mm, vias 60 -> 0
- net 3HardSyncIn3: track 95.7 -> 0.00 mm, vias 2 -> 0
- net 3VTO_1: track 93.2 -> 0.00 mm, vias 6 -> 0
- net Net-(C106-Pad1): track 90.3 -> 0.00 mm, vias 6 -> 0
- net Net-(C107-Pad1): track 82.3 -> 0.00 mm, vias 2 -> 0
- net Net-(R127-Pad2): track 77.2 -> 0.00 mm, vias 4 -> 0
- net 3PWM_In5: track 67.7 -> 0.00 mm
- net +5V: track 62.7 -> 0.00 mm, vias 3 -> 0
- net 3Octave: track 59.1 -> 0.00 mm, vias 2 -> 0
- net 3FM_Lin_In4: track 54.0 -> 0.00 mm, vias 4 -> 0
- net Net-(R151-Pad1): track 52.1 -> 0.00 mm, vias 4 -> 0
- net Net-(D103-Pad2): track 44.7 -> 0.00 mm
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