File: KicadJE_Util_RevA/KicadJE_Util.kicad_pcb (KiCad board)
At the start: 2 copper layers, 268.5 x 128 mm, 248 parts, among them J101 Out1, J102 Out2, J103 In1.1, J104 In1.2, J105 In1.3, J106 In1.4, J201 Out2.1, J202 Out2.2, J203 In2.1, J204 CV2.1, J205 In2.2, J206 CV2.2, J301 In3.1, J302 Out3.1, J303 Out3.2, P101 HEADER_2x5_Doepfer, P201 HEADER_2x5_Doepfer, P301 HEADER_2x5_Doepfer, U101 TL072, U102 TL072, U201 TL072, U202 TL072, U301 TL072, U302 TL072

Commit message: Labels and DRC
Parts:
- removed the G*** at (249.5, 156.0)
- removed the H102 at (246.0, 39.0)
- removed the H103 at (246.0, 161.0)
- removed H201: ON, AJ:LED_Hole_3mm
- removed H202, H203, H204, H205, H302, H303, H304, H305: MountingHole_Pad, AJ:MountingHole_Eurorack3
- removed the H301 at (249.5, 51.0)
- removed TP101, TP201: Tri, AJ:Jack_6m3
- removed TP104, TP204: In2, AJ:Jack_6m3
- removed the TP106 at (48.3, -5.51)
- removed the TP108 at (50.8, -19.1)
- removed TP109: Gain2, AJ:Pot_6m3_scale1
- removed TP110: Gain1, AJ:Pot_6m3_scale1
- removed TP202: SQ, AJ:Jack_6m3
- removed TP203: In1, AJ:Jack_6m3
- removed TP205: In3, AJ:Jack_6m3
- removed TP206: SS, AJ:Jack_6m3
- removed TP207: Glide1, AJ:Pot_6m3_scale1
- removed TP208: Glide2, AJ:Pot_6m3_scale1
- removed the TP301 at (249.5, 115.0)
- removed the TP302 at (249.5, 135.0)
- removed the TP303 at (249.5, 145.0)
- removed the TP304 at (249.5, 65.0)
- removed the TP305 at (249.5, 85.0)
- added G***: LOGO, AJ:Johansen_engineering_logo_20mm, F.Cu at (132.0, 135.0)
- added G***: LOGO, AJ:Johansen_engineering_logo_20mm, F.Cu at (70.0, 135.0)
- R216, R217, R228, R229: footprint OptoDevice:R_LDR_10x8.5mm_P7.6mm_Vertical -> OptoDevice:R_LDR_5.0x4.1mm_P3mm_Vertical
- moved C209 135.7 mm to (127.8, 70.0)
- moved TP209 130.5 mm to (129.8, 90.5)
- moved R217 129.6 mm to (137.8, 100.0)
- moved TP210 129.6 mm to (148.5, 90.5)
- moved R216 129.5 mm to (119.0, 100.0)
- moved R225 127.6 mm to (143.5, 70.0), turned to 180 degrees
- moved R223 125.1 mm to (139.5, 70.0), turned to 180 degrees
- moved R222 124.2 mm to (120.0, 70.0), turned to 180 degrees
- moved C203 120.6 mm to (119.5, 84.8), turned to 90 degrees
- moved R229 120.5 mm to (143.2, 100.0)
- moved R228 120.4 mm to (127.2, 100.0), turned to 180 degrees
- moved D207 120.4 mm to (140.5, 104.8)
- moved D205 120.3 mm to (122.0, 104.8)
- moved R224 115.9 mm to (123.7, 70.0), turned to 180 degrees
- moved R226 115.5 mm to (124.5, 77.0), turned to 90 degrees
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Routing:
- net +12VA: track 233.9 -> 370.8 mm, vias 3 -> 5
- net -12VA: track 228.0 -> 320.5 mm
- net Net-(R204-Pad1): track 0.00 -> 85.9 mm
- net GND: track 128.9 -> 209.9 mm, vias 62 -> 86
- net Net-(R205-Pad1): track 0.00 -> 69.2 mm
- net Out2.1: track 0.00 -> 29.7 mm, vias 0 -> 2
- net Out2.2: track 0.00 -> 28.3 mm
- net Net-(D207-Pad2): track 0.00 -> 27.5 mm
- net In2.2: track 0.00 -> 25.1 mm, vias 0 -> 2
- net Net-(D205-Pad2): track 0.00 -> 22.9 mm
- net In2.1: track 0.00 -> 22.0 mm
- net Net-(C208-Pad1): track 0.00 -> 19.9 mm
- net Net-(C207-Pad1): track 0.00 -> 19.2 mm
- net Net-(R215-Pad1): track 0.00 -> 18.5 mm
- net Net-(R213-Pad1): track 0.00 -> 18.2 mm
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Other:
- board size 268.5 x 128 mm -> 242 x 128 mm
- board text added: "CV Util"
- board text added: "CV Util Rev A 22/03-2020 Johansen Engineering"
- board text added: "JLCJLCJLCJLC"
- board text added: "Johansen Engineering Glide Rev A 22/03-2020"
- board text removed: "3340"
- board text removed: "JE - AS3340 Rev A 07/03-2020"
