File: KicadJE_Util_RevA/KicadJE_Util_Faceplate_Generic.kicad_pcb (KiCad board)
At the start: 2 copper layers, 40 x 128 mm, 16 parts

Commit message: Generic Face Gerber
Parts:
- added TP103: In1, AJ:Jack_6m3, F.Cu at (121.0, 135.0)
- added TP108: PWM, AJ:Jack_6m3, F.Cu at (101.0, 135.0)
Other:
- board text added: "1"
- board text added: "2"
- board text added: "8U"
- board text added: "Generic Faceplate Rev A 28/04-2020 Johansen Engineering"
- board text removed: "CV"
- board text removed: "CV Util Rev A 22/03-2020 Johansen Engineering"
- board text removed: "Gain1"
- board text removed: "Gain2"
- board text removed: "In1"
- board text removed: "In2"
- board text removed: "Inv1"
- board text removed: "Inv2"
- board text removed: "Offset1"
- board text removed: "Offset2"
Changed lines of the file:
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@@
   (general
     (thickness 1.6)
-    (drawings 49)
+    (drawings 66)
     (tracks 0)
     (zones 0)
-    (modules 16)
+    (modules 18)
     (nets 2)
   )
@@
       (drillshape 0)
       (scaleselection 1)
-      (outputdirectory "GerberRevA"))
+      (outputdirectory "GerberRevA_GenericFace"))
   )
   (net 0 "")
@@
     (uvia_drill 0.1)
     (add_net GND)
+  )
+  (module AJ:Jack_6m3 (layer F.Cu)
+    (at 121 135)
+    (descr "Mounting Hole 6.5mm, no annular")
+    (tags "mounting hole 6.5mm no annular")
+    (attr virtual)
+    (fp_text reference TP103 (at 0 0) (layer F.SilkS) hide
+      (effects (font (size 1 1) (thickness 0.15)))
+    )
+    (fp_text value In1 (at 0 0) (layer F.Fab)
+      (effects (font (size 1 1) (thickness 0.15)))
+    )
+    (fp_text user %R (at 0.3 0) (layer F.Fab)
+      (effects (font (size 1 1) (thickness 0.15)))
+    )
+    (fp_circle (center 0 0) (end 4.5 0) (layer Cmts.User) (width 0.15))
+    (fp_circle (center 0 0) (end 5 0) (layer F.CrtYd) (width 0.05))
+    (pad 1 thru_hole circle (at 0 0) (size 6.5 6.5) (drill 6.3) (layers *.Cu *.Mask)
+      (net 1 GND))
+  )
+  (module AJ:Jack_6m3 (layer F.Cu)
+    (at 101 135)
+    (descr "Mounting Hole 6.5mm, no annular")
+    (tags "mounting hole 6.5mm no annular")
+    (attr virtual)
+    (fp_text reference TP108 (at 0 0) (layer F.SilkS) hide
+      (effects (font (size 1 1) (thickness 0.15)))
+    )
+    (fp_text value PWM (at 0 0) (layer F.Fab)
+      (effects (font (size 1 1) (thickness 0.15)))
+    )
+    (fp_text user %R (at 0.3 0) (layer F.Fab)
+      (effects (font (size 1 1) (thickness 0.15)))
+    )
+    (fp_circle (center 0 0) (end 4.5 0) (layer Cmts.User) (width 0.15))
+    (fp_circle (center 0 0) (end 5 0) (layer F.CrtYd) (width 0.05))
+    (pad 1 thru_hole circle (at 0 0) (size 6.5 6.5) (drill 6.3) (layers *.Cu *.Mask)
+      (net 1 GND))
   )
   (module AJ:Pot_6m3_scale1 (layer F.Cu)
@@
     (pad "" np_thru_hole circle (at 0 0) (size 3 3) (drill 3) (layers *.Cu *.Mask))
   )
+  (gr_line (start 97 110) (end 95 110) (layer F.SilkS) (width 0.12))
+  (gr_line (start 101 115) (end 97 110) (layer F.SilkS) (width 0.12))
+  (gr_line (start 97 120) (end 95 120) (layer F.SilkS) (width 0.12))
+  (gr_line (start 101 125) (end 97 120) (layer F.SilkS) (width 0.12))
+  (gr_line (start 125 130) (end 126.5 130) (layer F.SilkS) (width 0.12))
+  (gr_line (start 121 135) (end 125 130) (layer F.SilkS) (width 0.12))
+  (gr_line (start 125 120) (end 126.5 120) (layer F.SilkS) (width 0.12))
+  (gr_line (start 121 125) (end 125 120) (layer F.SilkS) (width 0.12))
+  (gr_poly (pts (xy 116 148) (xy 106 148) (xy 106 142) (xy 116 142)) (layer F.SilkS) (width 0.1))
+  (gr_poly (pts (xy 116 138) (xy 106 138) (xy 106 132) (xy 116 132)) (layer F.SilkS) (width 0.1))
+  (gr_poly (pts (xy 116 128) (xy 106 128) (xy 106 122) (xy 116 122)) (layer F.SilkS) (width 0.1))
+  (gr_poly (pts (xy 129 105) (xy 93 105) (xy 93 93) (xy 129 93)) (layer F.SilkS) (width 0.1))
+  (gr_poly (pts (xy 116 118) (xy 106 118) (xy 106 112) (xy 116 112)) (layer F.SilkS) (width 0.1))
+  (gr_poly (pts (xy 99 77) (xy 92 77) (xy 92 73) (xy 99 73)) (layer F.SilkS) (width 0.1))
+  (gr_poly (pts (xy 130 77) (xy 123 77) (xy 123 73) (xy 130 73)) (layer F.SilkS) (width 0.1))
+  (gr_poly (pts (xy 130 57) (xy 123 57) (xy 123 53) (xy 130 53)) (layer F.SilkS) (width 0.1))
+  (gr_poly (pts (xy 99 57) (xy 92 57) (xy 92 53) (xy 99 53)) (layer F.SilkS) (width 0.1))
+  (gr_circle (center 121 135) (end 117.75 135.5) (layer Dwgs.User) (width 0.15))
+  (gr_circle (center 101 135) (end 97.75 135.5) (layer Dwgs.User) (width 0.15))
+  (gr_line (start 97 130) (end 95 130) (layer F.SilkS) (width 0.12))
+  (gr_line (start 101 135) (end 97 130) (layer F.SilkS) (width 0.12))
+  (gr_text 1 (at 94 130) (layer F.SilkS)
+    (effects (font (size 3 2) (thickness 0.5)))
+  )
+  (gr_text 2 (at 127.5 130) (layer F.SilkS)
+    (effects (font (size 3 2) (thickness 0.5)))
+  )
   (gr_text JLCJLCJLCJLC (at 92 158.5 90) (layer B.SilkS)
     (effects (font (size 1 1) (thickness 0.1)) (justify mirror))
   )
-  (gr_text "CV Util Rev A\n22/03-2020\nJohansen Engineering" (at 111 152.5) (layer B.SilkS)
+  (gr_text "Generic Faceplate Rev A\n28/04-2020\nJohansen Engineering" (at 111 152.5) (layer B.SilkS)
     (effects (font (size 1.3 1.2) (thickness 0.3)) (justify mirror))
   )
-  (gr_text Gain1 (at 101 75) (layer F.SilkS)
-    (effects (font (size 3 2) (thickness 0.5)))
-  )
-  (gr_text Offset1 (at 101 55) (layer F.SilkS)
+  (gr_text 1 (at 101 75) (layer F.SilkS)
+    (effects (font (size 3 2) (thickness 0.5)))
+  )
+  (gr_text 1 (at 101 55) (layer F.SilkS)
     (effects (font (size 3 2) (thickness 0.5)))
   )
@@
   (gr_line (start 121 57.5) (end 121 145) (layer F.SilkS) (width 0.12))
   (gr_line (start 101 145) (end 101 65.5) (layer F.SilkS) (width 0.12))
-  (gr_line (start 121 115) (end 127.5 115) (layer F.SilkS) (width 0.12))
-  (gr_line (start 127.5 115) (end 127.5 112) (layer F.SilkS) (width 0.12))
-  (gr_line (start 121 125) (end 127.5 125) (layer F.SilkS) (width 0.12))
-  (gr_line (start 127.5 125) (end 127.5 122) (layer F.SilkS) (width 0.12))
+  (gr_line (start 121 115) (end 125 110) (layer F.SilkS) (width 0.12))
+  (gr_line (start 125 110) (end 126.5 110) (layer F.SilkS) (width 0.12))
   (gr_line (start 127.5 145) (end 127.5 142) (layer F.SilkS) (width 0.12))
   (gr_line (start 121 145) (end 127.5 145) (layer F.SilkS) (width 0.12))
   (gr_line (start 94 145) (end 94 142) (layer F.SilkS) (width 0.12))
   (gr_line (start 101 145) (end 94 145) (layer F.SilkS) (width 0.12))
-  (gr_line (start 94 125) (end 94 122) (layer F.SilkS) (width 0.12))
-  (gr_line (start 101 125) (end 94 125) (layer F.SilkS) (width 0.12))
-  (gr_line (start 101 115) (end 94 115) (layer F.SilkS) (width 0.12))
-  (gr_line (start 94 115) (end 94 112) (layer F.SilkS) (width 0.12))
-  (gr_text Inv1 (at 94 120) (layer F.SilkS)
+  (gr_text 1 (at 94 120) (layer F.SilkS)
     (effects (font (size 3 2) (thickness 0.5)))
   )
@@
     (effects (font (size 3 2) (thickness 0.5)))
   )
-  (gr_text In1 (at 94 110) (layer F.SilkS)
+  (gr_text 1 (at 94 110) (layer F.SilkS)
     (effects (font (size 3 2) (thickness 0.5)))
   )
@@
     (effects (font (size 3 2) (thickness 0.5)))
   )
-  (gr_text Inv2 (at 127.5 120) (layer F.SilkS)
-    (effects (font (size 3 2) (thickness 0.5)))
-  )
-  (gr_text In2 (at 127.5 110) (layer F.SilkS)
-    (effects (font (size 3 2) (thickness 0.5)))
-  )
-  (gr_text Gain2 (at 121 75) (layer F.SilkS)
-    (effects (font (size 3 2) (thickness 0.5)))
-  )
-  (gr_text Offset2 (at 121 55) (layer F.SilkS)
+  (gr_text 2 (at 127.5 120) (layer F.SilkS)
+    (effects (font (size 3 2) (thickness 0.5)))
+  )
+  (gr_text 2 (at 127.5 110) (layer F.SilkS)
+    (effects (font (size 3 2) (thickness 0.5)))
+  )
+  (gr_text 2 (at 121 75) (layer F.SilkS)
+    (effects (font (size 3 2) (thickness 0.5)))
+  )
+  (gr_text 2 (at 121 55) (layer F.SilkS)
     (effects (font (size 3 2) (thickness 0.5)))
   )
@@
   (gr_line (start 111 50) (end 111 150) (layer Dwgs.User) (width 0.15))
   (gr_line (start 101 150) (end 101 50) (layer Dwgs.User) (width 0.15))
-  (gr_text CV (at 111 40.5) (layer F.SilkS)
+  (gr_text 8U (at 111 40.5) (layer F.SilkS)
     (effects (font (size 6 4) (thickness 1)))
   )
