File: KicadJE_Util_RevB/KicadJE_Util.sch (KiCad schematic (older format))
At the start: 78 parts, among them J101 Out1, J102 Out2, J103 In1.1, J104 In1.2, J105 In1.3, J106 In1.4, P101 HEADER_2x5_Doepfer, U101 TL072, U102 TL072

Commit message: input changed
Parts:
- added R?: 10k, Resistor_SMD:R_0805_2012Metric_Pad1.15x1.40mm_HandSolder, symbol Device:R
Connections:
- net GND: now also R?.1; no longer J103.TN, J104.TN, J105.TN, J106.TN
- new net: J103.TN, J104.TN, J105.TN, J106.TN, R?.2
Changed lines of the file:
@@
 Wire Wire Line
 	2125 2550 2025 2550
-Wire Wire Line
-	1975 2750 2125 2750
-Wire Wire Line
-	2125 2750 2125 2550
-Wire Wire Line
-	1975 3275 2125 3275
-Wire Wire Line
-	2125 3275 2125 3075
 $Comp
 L Connector:AudioJack2_SwitchT J106
@@
 Wire Wire Line
 	1975 4025 2225 4025
-Wire Wire Line
-	1975 4125 2125 4125
 Connection ~ 2125 3925
-Wire Wire Line
-	2125 3925 2125 4125
 Wire Wire Line
 	1975 3925 2025 3925
@@
 	0    1    1    0
 $EndComp
-Wire Wire Line
-	1975 4650 2125 4650
 Wire Wire Line
 	2375 5325 2425 5325
@@
 	1    0    0    -1
 $EndComp
-Wire Wire Line
-	2125 4125 2125 4450
-Connection ~ 2125 4125
 $Comp
 L Device:R R110
@@
 	0    1    1    0
 $EndComp
-Wire Wire Line
-	2125 3275 2125 3925
-Connection ~ 2125 3275
-Connection ~ 2125 2750
-Connection ~ 2125 4650
 $Comp
 L power:-12VA #PWR?
@@
 	1    0    0    -1
 $EndComp
-Wire Wire Line
-	2125 2750 2125 3075
 Connection ~ 2125 3075
 Text GLabel 3375 2650 2    50   Input ~ 0
@@
 Text Notes 7450 5200 0    97   ~ 0
 CHECK POTS
+$Comp
+L Device:R R?
+U 1 1 5EA9C392
+P 2375 3550
+AR Path="/5EA9C392" Ref="R?"  Part="1"
+AR Path="/5C8C5FC0/5EA9C392" Ref="R?"  Part="1"
+AR Path="/5CAAE8D3/5EA9C392" Ref="R?"  Part="1"
+AR Path="/5E4B0DD9/5EA9C392" Ref="R?"  Part="1"
+AR Path="/5F49A670/5EA9C392" Ref="R?"  Part="1"
+F 0 "R?" V 2300 3550 50  0000 C CNN
+F 1 "10k" V 2375 3550 50  0000 C CNN
+F 2 "Resistor_SMD:R_0805_2012Metric_Pad1.15x1.40mm_HandSolder" V 2305 3550 50  0001 C CNN
+F 3 "~" H 2375 3550 50  0001 C CNN
+	1    2375 3550
+	0    1    1    0
+$EndComp
+Wire Wire Line
+	2225 3550 2175 3550
+Wire Wire Line
+	2175 3550 2175 3275
+Wire Wire Line
+	1975 2750 2175 2750
+Wire Wire Line
+	2125 2550 2125 3075
+Connection ~ 2175 3275
+Wire Wire Line
+	2175 3275 2175 2750
+Wire Wire Line
+	1975 3275 2175 3275
+Wire Wire Line
+	2125 3075 2125 3725
+Wire Wire Line
+	2175 3550 2175 4125
+Connection ~ 2175 3550
+Wire Wire Line
+	2175 4650 2175 4125
+Connection ~ 2175 4125
+Wire Wire Line
+	1975 4650 2175 4650
+Wire Wire Line
+	1975 4125 2175 4125
+Wire Wire Line
+	2125 3925 2125 4450
+Wire Wire Line
+	2525 3550 2575 3550
+Wire Wire Line
+	2575 3550 2575 3725
+Wire Wire Line
+	2575 3725 2125 3725
+Connection ~ 2125 3725
+Wire Wire Line
+	2125 3725 2125 3925
 $EndSCHEMATC

Commit message: attempt to go to Kicad 7
Parts:
- P101: symbol Eurorack:HEADER_2x5_Doepfer -> KicadJE_Util-rescue:HEADER_2x5_Doepfer-Eurorack
- RV101, RV102, RV103, RV104: symbol Envelope-cache-2018-08-04-13-00-04:POT -> KicadJE_Util-rescue:POT-Envelope-cache-2018-08-04-13-00-04
Changed lines of the file:
@@
 $EndComp
 $Comp
-L Envelope-cache-2018-08-04-13-00-04:GND #PWR0101
+L KicadJE_Util-rescue:GND-Envelope-cache-2018-08-04-13-00-04 #PWR0101
 U 1 1 5F4B92B1
 P 1550 6200
@@
 $EndComp
 $Comp
-L Eurorack:HEADER_2x5_Doepfer P?
+L KicadJE_Util-rescue:HEADER_2x5_Doepfer-Eurorack P?
 U 1 1 5F4F8A1B
 P 1875 1400
@@
 $EndComp
 $Comp
-L Envelope-cache-2018-08-04-13-00-04:GND #PWR0105
+L KicadJE_Util-rescue:GND-Envelope-cache-2018-08-04-13-00-04 #PWR0105
 U 1 1 5F4F8A5B
 P 2275 1400
@@
 $EndComp
 $Comp
-L Envelope-cache-2018-08-04-13-00-04:GND #PWR0102
+L KicadJE_Util-rescue:GND-Envelope-cache-2018-08-04-13-00-04 #PWR0102
 U 1 1 5F4F8A76
 P 1625 1400
@@
 Connection ~ 2975 2075
 $Comp
-L Envelope-cache-2018-08-04-13-00-04:GND #PWR0111
+L KicadJE_Util-rescue:GND-Envelope-cache-2018-08-04-13-00-04 #PWR0111
 U 1 1 5EF57B05
 P 2850 2075
@@
 	2850 2075 2975 2075
 $Comp
-L Envelope-cache-2018-08-04-13-00-04:GND #PWR0118
+L KicadJE_Util-rescue:GND-Envelope-cache-2018-08-04-13-00-04 #PWR0118
 U 1 1 5EF95D3D
 P 3500 7150
@@
 Connection ~ 3000 4025
 $Comp
-L Envelope-cache-2018-08-04-13-00-04:GND #PWR0104
+L KicadJE_Util-rescue:GND-Envelope-cache-2018-08-04-13-00-04 #PWR0104
 U 1 1 5F094B26
 P 2125 4650
@@
 $EndComp
 $Comp
-L Envelope-cache-2018-08-04-13-00-04:GND #PWR0122
+L KicadJE_Util-rescue:GND-Envelope-cache-2018-08-04-13-00-04 #PWR0122
 U 1 1 5F665D87
 P 5375 6025
@@
 $EndComp
 $Comp
-L Envelope-cache-2018-08-04-13-00-04:GND #PWR0120
+L KicadJE_Util-rescue:GND-Envelope-cache-2018-08-04-13-00-04 #PWR0120
 U 1 1 5F666F6F
 P 5375 5025
@@
 $EndComp
 $Comp
-L Envelope-cache-2018-08-04-13-00-04:GND #PWR0119
+L KicadJE_Util-rescue:GND-Envelope-cache-2018-08-04-13-00-04 #PWR0119
 U 1 1 5F87AA0C
 P 5375 4275
@@
 $EndComp
 $Comp
-L Envelope-cache-2018-08-04-13-00-04:GND #PWR0121
+L KicadJE_Util-rescue:GND-Envelope-cache-2018-08-04-13-00-04 #PWR0121
 U 1 1 5F8D7E2C
 P 5375 5275
@@
 Flow2
 $Comp
-L Envelope-cache-2018-08-04-13-00-04:POT RV?
+L KicadJE_Util-rescue:POT-Envelope-cache-2018-08-04-13-00-04 RV?
 U 1 1 60D4C6A7
 P 3325 7100
@@
 $EndComp
 $Comp
-L Envelope-cache-2018-08-04-13-00-04:GND #PWR0125
+L KicadJE_Util-rescue:GND-Envelope-cache-2018-08-04-13-00-04 #PWR0125
 U 1 1 5FA1508D
 P 6475 7125
@@
 $EndComp
 $Comp
-L Envelope-cache-2018-08-04-13-00-04:POT RV?
+L KicadJE_Util-rescue:POT-Envelope-cache-2018-08-04-13-00-04 RV?
 U 1 1 5FA15097
 P 6300 7075
@@
 	4500 6525 4500 525
 $Comp
-L Envelope-cache-2018-08-04-13-00-04:POT RV?
+L KicadJE_Util-rescue:POT-Envelope-cache-2018-08-04-13-00-04 RV?
 U 1 1 5FBFC8B7
 P 6275 5000
@@
 	6650 5675 6650 5600
 $Comp
-L Envelope-cache-2018-08-04-13-00-04:POT RV?
+L KicadJE_Util-rescue:POT-Envelope-cache-2018-08-04-13-00-04 RV?
 U 1 1 5FC00159
 P 6275 6000
@@
 $EndComp
 $Comp
-L Envelope-cache-2018-08-04-13-00-04:GND #PWR0126
+L KicadJE_Util-rescue:GND-Envelope-cache-2018-08-04-13-00-04 #PWR0126
 U 1 1 5FCDB135
 P 6750 6100
@@
 $EndComp
 $Comp
-L Envelope-cache-2018-08-04-13-00-04:GND #PWR0127
+L KicadJE_Util-rescue:GND-Envelope-cache-2018-08-04-13-00-04 #PWR0127
 U 1 1 5FD07A67
 P 6775 5125
