File: KicadJE_Util_RevB/KicadJE_Util_CV2.sch (KiCad schematic (older format))
At the start: 76 parts, among them J201 Out2.1, J202 Out2.2, J203 In2.1, J204 CV2.1, J205 In2.2, J206 CV2.2, P201 HEADER_2x5_Doepfer, U201 TL072, U202 TL072

Commit message: input changed
Parts:
- added R?: 10k, Resistor_SMD:R_0805_2012Metric_Pad1.15x1.40mm_HandSolder, symbol Device:R
- C208: value 1u -> Open
- C212: value OPEN -> 4u7
- R217: value LDR03_In2 -> OPEN
- R223: value 680R -> OPEN
- R225: value OPEN -> 680R
- R229: value OPEN -> LDR03_In2
Connections:
- net GND: now also R?.1; no longer J203.TN, J204.TN, J205.TN, J206.TN
- new net: J203.TN, J204.TN, J205.TN, J206.TN, R?.2
Changed lines of the file:
@@
 	2175 2550 2075 2550
 Wire Wire Line
-	2025 2750 2175 2750
-Wire Wire Line
 	2175 2750 2175 2550
 Wire Wire Line
-	2025 3275 2175 3275
+	2025 3275 2050 3275
 Wire Wire Line
 	2175 3275 2175 3075
@@
 Wire Wire Line
 	2025 4025 2275 4025
-Wire Wire Line
-	2025 4125 2175 4125
 Connection ~ 2175 3925
 Wire Wire Line
@@
 	0    1    1    0
 $EndComp
-Wire Wire Line
-	2025 4650 2175 4650
 $Comp
 L Device:R R?
@@
 	4450 4850 575  4850
 Wire Wire Line
-	2175 3275 2175 3925
+	2175 3275 2175 3600
 Wire Wire Line
 	3050 2650 3050 2750
@@
 Wire Wire Line
 	3050 4025 3050 4125
-Wire Wire Line
-	2175 4125 2725 4125
 $Comp
 L Amplifier_Operational:TL072 U?
@@
 AR Path="/5F49A670/5E9CE478" Ref="R?"  Part="1"
 AR Path="/5FDBD837/5E9CE478" Ref="R215"  Part="1"
-F 0 "R215" V 4925 3300 50  0000 C CNN
+F 0 "R215" V 4925 3375 50  0000 C CNN
 F 1 "20k" V 5025 3375 50  0000 C CNN
 F 2 "Resistor_SMD:R_0805_2012Metric_Pad1.15x1.40mm_HandSolder" V 4955 3375 50  0001 C CNN
@@
 AR Path="/5F49A670/5E9CE47E" Ref="R?"  Part="1"
 AR Path="/5FDBD837/5E9CE47E" Ref="R213"  Part="1"
-F 0 "R213" V 4925 1475 50  0000 C CNN
+F 0 "R213" V 4950 1550 50  0000 C CNN
 F 1 "20k" V 5025 1550 50  0000 C CNN
 F 2 "Resistor_SMD:R_0805_2012Metric_Pad1.15x1.40mm_HandSolder" V 4955 1550 50  0001 C CNN
@@
 AR Path="/5F49A670/5E9CE4AF" Ref="R?"  Part="1"
 AR Path="/5FDBD837/5E9CE4AF" Ref="R212"  Part="1"
-F 0 "R212" V 4925 725 50  0000 C CNN
+F 0 "R212" V 4925 800 50  0000 C CNN
 F 1 "20k" V 5025 800 50  0000 C CNN
 F 2 "Resistor_SMD:R_0805_2012Metric_Pad1.15x1.40mm_HandSolder" V 4955 800 50  0001 C CNN
@@
 AR Path="/5F49A670/5E9CE4C1" Ref="R?"  Part="1"
 AR Path="/5FDBD837/5E9CE4C1" Ref="R214"  Part="1"
-F 0 "R214" V 4925 2550 50  0000 C CNN
+F 0 "R214" V 4925 2625 50  0000 C CNN
 F 1 "20k" V 5025 2625 50  0000 C CNN
 F 2 "Resistor_SMD:R_0805_2012Metric_Pad1.15x1.40mm_HandSolder" V 4955 2625 50  0001 C CNN
@@
 AR Path="/5F49A670/5E9CE4D3" Ref="R?"  Part="1"
 AR Path="/5FDBD837/5E9CE4D3" Ref="R221"  Part="1"
-F 0 "R221" V 6025 2900 50  0000 C CNN
+F 0 "R221" V 6025 2975 50  0000 C CNN
 F 1 "220R" V 6125 2975 50  0000 C CNN
 F 2 "Resistor_SMD:R_0805_2012Metric_Pad1.15x1.40mm_HandSolder" V 6055 2975 50  0001 C CNN
@@
 AR Path="/5F49A670/5E9CE4EB" Ref="R?"  Part="1"
 AR Path="/5FDBD837/5E9CE4EB" Ref="R224"  Part="1"
-F 0 "R224" V 6725 1225 50  0000 C CNN
+F 0 "R224" V 6725 1300 50  0000 C CNN
 F 1 "OPEN" V 6825 1300 50  0000 C CNN
 F 2 "Resistor_SMD:R_0805_2012Metric_Pad1.15x1.40mm_HandSolder" V 6755 1300 50  0001 C CNN
@@
 AR Path="/5F49A670/5E9CE4F1" Ref="R?"  Part="1"
 AR Path="/5FDBD837/5E9CE4F1" Ref="R222"  Part="1"
-F 0 "R222" V 6325 1225 50  0000 C CNN
+F 0 "R222" V 6325 1300 50  0000 C CNN
 F 1 "680R" V 6425 1300 50  0000 C CNN
 F 2 "Resistor_SMD:R_0805_2012Metric_Pad1.15x1.40mm_HandSolder" V 6355 1300 50  0001 C CNN
@@
 AR Path="/5F49A670/5E9CE501" Ref="R?"  Part="1"
 AR Path="/5FDBD837/5E9CE501" Ref="R225"  Part="1"
-F 0 "R225" V 6800 3050 50  0000 C CNN
-F 1 "OPEN" V 6900 3125 50  0000 C CNN
+F 0 "R225" V 6825 3125 50  0000 C CNN
+F 1 "680R" V 6900 3125 50  0000 C CNN
 F 2 "Resistor_SMD:R_0805_2012Metric_Pad1.15x1.40mm_HandSolder" V 6830 3125 50  0001 C CNN
 F 3 "~" H 6900 3125 50  0001 C CNN
@@
 AR Path="/5F49A670/5E9CE507" Ref="R?"  Part="1"
 AR Path="/5FDBD837/5E9CE507" Ref="R223"  Part="1"
-F 0 "R223" V 6400 3050 50  0000 C CNN
-F 1 "680R" V 6500 3125 50  0000 C CNN
+F 0 "R223" V 6425 3100 50  0000 C CNN
+F 1 "OPEN" V 6500 3125 50  0000 C CNN
 F 2 "Resistor_SMD:R_0805_2012Metric_Pad1.15x1.40mm_HandSolder" V 6430 3125 50  0001 C CNN
 F 3 "~" H 6500 3125 50  0001 C CNN
@@
 AR Path="/5FDBD837/5E9CE52F" Ref="TP209"  Part="1"
 F 0 "TP209" H 7708 1268 50  0000 L CNN
-F 1 "Flow1" H 7708 1177 50  0000 L CNN
+F 1 "Flow1" H 7700 1350 50  0000 L CNN
 F 2 "TestPoint:TestPoint_THTPad_2.0x2.0mm_Drill1.0mm" H 7850 1150 50  0001 C CNN
 F 3 "~" H 7850 1150 50  0001 C CNN
@@
 AR Path="/5FDBD837/5E9CE537" Ref="TP210"  Part="1"
 F 0 "TP210" H 8033 3093 50  0000 L CNN
-F 1 "Flow2" H 8033 3002 50  0000 L CNN
+F 1 "Flow2" H 8050 3175 50  0000 L CNN
 F 2 "TestPoint:TestPoint_THTPad_2.0x2.0mm_Drill1.0mm" H 8175 2975 50  0001 C CNN
 F 3 "~" H 8175 2975 50  0001 C CNN
@@
 Wire Wire Line
 	3025 4550 3025 4650
-Wire Wire Line
-	2175 4650 3025 4650
 $Comp
 L Device:R R?
@@
 AR Path="/5EC49EEF" Ref="C?"  Part="1"
 AR Path="/5FDBD837/5EC49EEF" Ref="C210"  Part="1"
-F 0 "C210" H 7100 3500 50  0000 L CNN
-F 1 "1u" H 7075 3250 50  0000 L CNN
+F 0 "C210" H 7175 3475 50  0000 L CNN
+F 1 "1u" H 7175 3275 50  0000 L CNN
 F 2 "Capacitor_SMD:C_0805_2012Metric_Pad1.15x1.40mm_HandSolder" H 7188 3225 50  0001 C CNN
 F 3 "~" H 7150 3375 50  0001 C CNN
@@
 AR Path="/5F49A670/5ECE138C" Ref="R?"  Part="1"
 AR Path="/5FDBD837/5ECE138C" Ref="R220"  Part="1"
-F 0 "R220" V 6000 1075 50  0000 C CNN
+F 0 "R220" V 6000 1150 50  0000 C CNN
 F 1 "220R" V 6100 1150 50  0000 C CNN
 F 2 "Resistor_SMD:R_0805_2012Metric_Pad1.15x1.40mm_HandSolder" V 6030 1150 50  0001 C CNN
@@
 AR Path="/5ED09A02" Ref="C?"  Part="1"
 AR Path="/5FDBD837/5ED09A02" Ref="C211"  Part="1"
-F 0 "C211" H 7600 1975 50  0000 L CNN
-F 1 "4u7" H 7575 1725 50  0000 L CNN
+F 0 "C211" H 7650 1925 50  0000 L CNN
+F 1 "4u7" H 7675 1750 50  0000 L CNN
 F 2 "Capacitor_SMD:C_0805_2012Metric_Pad1.15x1.40mm_HandSolder" H 7688 1700 50  0001 C CNN
 F 3 "~" H 7650 1850 50  0001 C CNN
@@
 AR Path="/5F49A670/5ED74619" Ref="R?"  Part="1"
 AR Path="/5FDBD837/5ED74619" Ref="R219"  Part="1"
-F 0 "R219" V 5525 1475 50  0000 C CNN
+F 0 "R219" V 5700 1550 50  0000 C CNN
 F 1 "20k" V 5625 1550 50  0000 C CNN
 F 2 "Resistor_SMD:R_0805_2012Metric_Pad1.15x1.40mm_HandSolder" V 5555 1550 50  0001 C CNN
@@
 U 1 1 5EDE7551
 P 7750 3175
-F 0 "R229" V 7650 3050 50  0000 C CNN
-F 1 "OPEN" V 7750 3175 50  0000 C CNN
+F 0 "R229" H 7900 3125 50  0000 C CNN
+F 1 "LDR03_In2" H 8000 3225 50  0000 C CNN
 F 2 "OptoDevice:R_LDR_5.0x4.1mm_P3mm_Vertical" V 7925 3175 50  0001 C CNN
 F 3 "http://www.elektronica-componenten.nl/WebRoot/StoreNL/Shops/61422969/54F1/BA0C/C664/31B9/2173/C0A8/2AB9/2AEF/LDR03IMP.pdf" H 7750 3125 50  0001 C CNN
@@
 AR Path="/5F49A670/5EE03E4D" Ref="R?"  Part="1"
 AR Path="/5FDBD837/5EE03E4D" Ref="R218"  Part="1"
-F 0 "R218" V 5500 3300 50  0000 C CNN
+F 0 "R218" V 5700 3375 50  0000 C CNN
 F 1 "20k" V 5600 3375 50  0000 C CNN
 F 2 "Resistor_SMD:R_0805_2012Metric_Pad1.15x1.40mm_HandSolder" V 5530 3375 50  0001 C CNN
@@
 AR Path="/5EE0450C" Ref="C?"  Part="1"
 AR Path="/5FDBD837/5EE0450C" Ref="C212"  Part="1"
-F 0 "C212" V 7700 3625 50  0000 L CNN
-F 1 "OPEN" H 7850 3575 50  0000 L CNN
+F 0 "C212" H 7525 3425 50  0000 L CNN
+F 1 "4u7" H 7575 3600 50  0000 L CNN
 F 2 "Capacitor_SMD:C_0805_2012Metric_Pad1.15x1.40mm_HandSolder" H 7788 3350 50  0001 C CNN
 F 3 "~" H 7750 3500 50  0001 C CNN
@@
 U 1 1 5EE4B85A
 P 5475 1850
-F 0 "R216" V 5375 1725 50  0000 C CNN
+F 0 "R216" V 5550 1850 50  0000 C CNN
 F 1 "OPEN" V 5475 1850 50  0000 C CNN
 F 2 "OptoDevice:R_LDR_5.0x4.1mm_P3mm_Vertical" V 5650 1850 50  0001 C CNN
@@
 AR Path="/5F49A670/5EE6CEE9" Ref="R?"  Part="1"
 AR Path="/5FDBD837/5EE6CEE9" Ref="R227"  Part="1"
-F 0 "R227" V 7275 2900 50  0000 C CNN
+F 0 "R227" V 7475 2975 50  0000 C CNN
 F 1 "20k" V 7375 2975 50  0000 C CNN
 F 2 "Resistor_SMD:R_0805_2012Metric_Pad1.15x1.40mm_HandSolder" V 7305 2975 50  0001 C CNN
@@
 U 1 1 5EE915DB
 P 5475 3675
-F 0 "R217" V 5375 3550 50  0000 C CNN
-F 1 "LDR03_In2" V 5475 3675 50  0000 C CNN
+F 0 "R217" V 5550 3675 50  0000 C CNN
+F 1 "OPEN" V 5475 3675 50  0000 C CNN
 F 2 "OptoDevice:R_LDR_5.0x4.1mm_P3mm_Vertical" V 5650 3675 50  0001 C CNN
 F 3 "http://www.elektronica-componenten.nl/WebRoot/StoreNL/Shops/61422969/54F1/BA0C/C664/31B9/2173/C0A8/2AB9/2AEF/LDR03IMP.pdf" H 5475 3625 50  0001 C CNN
@@
 AR Path="/5EE915E5" Ref="C?"  Part="1"
 AR Path="/5FDBD837/5EE915E5" Ref="C208"  Part="1"
-F 0 "C208" V 5750 3800 50  0000 L CNN
-F 1 "1u" V 5900 3750 50  0000 L CNN
+F 0 "C208" V 5650 3575 50  0000 L CNN
+F 1 "Open" V 5925 3575 50  0000 L CNN
 F 2 "Capacitor_SMD:C_0805_2012Metric_Pad1.15x1.40mm_HandSolder" H 5838 3525 50  0001 C CNN
 F 3 "~" H 5800 3675 50  0001 C CNN
@@
 AR Path="/5EED43F0" Ref="C?"  Part="1"
 AR Path="/5FDBD837/5EED43F0" Ref="C209"  Part="1"
-F 0 "C209" H 6950 1975 50  0000 L CNN
-F 1 "1u" H 6925 1725 50  0000 L CNN
+F 0 "C209" H 7025 1925 50  0000 L CNN
+F 1 "1u" H 7025 1775 50  0000 L CNN
 F 2 "Capacitor_SMD:C_0805_2012Metric_Pad1.15x1.40mm_HandSolder" H 7038 1700 50  0001 C CNN
 F 3 "~" H 7000 1850 50  0001 C CNN
@@
 Wire Wire Line
 	2450 1000 2650 1000
+$Comp
+L Device:R R?
+U 1 1 5EA587F0
+P 1800 3600
+AR Path="/5EA587F0" Ref="R?"  Part="1"
+AR Path="/5C8C5FC0/5EA587F0" Ref="R?"  Part="1"
+AR Path="/5CAAE8D3/5EA587F0" Ref="R?"  Part="1"
+AR Path="/5E4B0DD9/5EA587F0" Ref="R?"  Part="1"
+AR Path="/5F49A670/5EA587F0" Ref="R?"  Part="1"
+AR Path="/5FDBD837/5EA587F0" Ref="R?"  Part="1"
+F 0 "R?" V 1725 3600 50  0000 C CNN
+F 1 "10k" V 1800 3600 50  0000 C CNN
+F 2 "Resistor_SMD:R_0805_2012Metric_Pad1.15x1.40mm_HandSolder" V 1730 3600 50  0001 C CNN
+F 3 "~" H 1800 3600 50  0001 C CNN
+	1    1800 3600
+	0    1    1    0
+$EndComp
+Wire Wire Line
+	2175 4650 3025 4650
+Wire Wire Line
+	2025 4650 2025 4800
+Wire Wire Line
+	2025 4800 1400 4800
+Wire Wire Line
+	1400 4800 1400 4250
+Wire Wire Line
+	1400 4250 2025 4250
+Wire Wire Line
+	2025 4125 2025 4250
+Wire Wire Line
+	2175 4125 2725 4125
+Wire Wire Line
+	1950 3600 2175 3600
+Connection ~ 2175 3600
+Wire Wire Line
+	2175 3600 2175 3925
+Wire Wire Line
+	2050 3275 2050 3475
+Wire Wire Line
+	2050 3475 1400 3475
+Wire Wire Line
+	1400 3475 1400 3600
+Connection ~ 1400 4250
+Wire Wire Line
+	1650 3600 1400 3600
+Connection ~ 1400 3600
+Wire Wire Line
+	1400 3600 1400 4250
+Wire Wire Line
+	2025 2750 2025 2900
+Wire Wire Line
+	2025 2900 1400 2900
+Wire Wire Line
+	1400 2900 1400 3475
+Connection ~ 1400 3475
 $EndSCHEMATC

Commit message: attempt to go to Kicad 7
Parts:
- P201: symbol Eurorack:HEADER_2x5_Doepfer -> KicadJE_Util-rescue:HEADER_2x5_Doepfer-Eurorack
- RV201, RV202: symbol Envelope-cache-2018-08-04-13-00-04:POT -> KicadJE_Util-rescue:POT-Envelope-cache-2018-08-04-13-00-04
Changed lines of the file:
@@
 $EndComp
 $Comp
-L Envelope-cache-2018-08-04-13-00-04:GND #PWR?
+L KicadJE_Util-rescue:GND-Envelope-cache-2018-08-04-13-00-04 #PWR?
 U 1 1 5E7BA3A7
 P 1600 6200
@@
 $EndComp
 $Comp
-L Eurorack:HEADER_2x5_Doepfer P?
+L KicadJE_Util-rescue:HEADER_2x5_Doepfer-Eurorack P?
 U 1 1 5E7BA3F7
 P 1925 1400
@@
 	2450 1050 2450 1000
 $Comp
-L Envelope-cache-2018-08-04-13-00-04:GND #PWR?
+L KicadJE_Util-rescue:GND-Envelope-cache-2018-08-04-13-00-04 #PWR?
 U 1 1 5E7BA42D
 P 2325 1400
@@
 $EndComp
 $Comp
-L Envelope-cache-2018-08-04-13-00-04:GND #PWR?
+L KicadJE_Util-rescue:GND-Envelope-cache-2018-08-04-13-00-04 #PWR?
 U 1 1 5E7BA43F
 P 1675 1400
@@
 Connection ~ 3025 2075
 $Comp
-L Envelope-cache-2018-08-04-13-00-04:GND #PWR?
+L KicadJE_Util-rescue:GND-Envelope-cache-2018-08-04-13-00-04 #PWR?
 U 1 1 5E7BA534
 P 2900 2075
@@
 Connection ~ 3050 4025
 $Comp
-L Envelope-cache-2018-08-04-13-00-04:GND #PWR?
+L KicadJE_Util-rescue:GND-Envelope-cache-2018-08-04-13-00-04 #PWR?
 U 1 1 5E7BA58B
 P 2175 4650
@@
 $EndComp
 $Comp
-L Envelope-cache-2018-08-04-13-00-04:GND #PWR?
+L KicadJE_Util-rescue:GND-Envelope-cache-2018-08-04-13-00-04 #PWR?
 U 1 1 5E9CE484
 P 4675 3400
@@
 $EndComp
 $Comp
-L Envelope-cache-2018-08-04-13-00-04:GND #PWR?
+L KicadJE_Util-rescue:GND-Envelope-cache-2018-08-04-13-00-04 #PWR?
 U 1 1 5E9CE48A
 P 4675 1575
@@
 $EndComp
 $Comp
-L Envelope-cache-2018-08-04-13-00-04:GND #PWR?
+L KicadJE_Util-rescue:GND-Envelope-cache-2018-08-04-13-00-04 #PWR?
 U 1 1 5E9CE4B5
 P 4675 825
@@
 $EndComp
 $Comp
-L Envelope-cache-2018-08-04-13-00-04:GND #PWR?
+L KicadJE_Util-rescue:GND-Envelope-cache-2018-08-04-13-00-04 #PWR?
 U 1 1 5E9CE4C7
 P 4675 2650
@@
 	4475 6525 4475 525
 $Comp
-L Envelope-cache-2018-08-04-13-00-04:POT RV?
+L KicadJE_Util-rescue:POT-Envelope-cache-2018-08-04-13-00-04 RV?
 U 1 1 5E9CE4DD
 P 6625 1150
@@
 $EndComp
 $Comp
-L Envelope-cache-2018-08-04-13-00-04:POT RV?
+L KicadJE_Util-rescue:POT-Envelope-cache-2018-08-04-13-00-04 RV?
 U 1 1 5E9CE4E5
 P 6700 2975
@@
 $EndComp
 $Comp
-L Envelope-cache-2018-08-04-13-00-04:GND #PWR?
+L KicadJE_Util-rescue:GND-Envelope-cache-2018-08-04-13-00-04 #PWR?
 U 1 1 5E9CE51D
 P 6700 3375
@@
 $EndComp
 $Comp
-L Envelope-cache-2018-08-04-13-00-04:GND #PWR?
+L KicadJE_Util-rescue:GND-Envelope-cache-2018-08-04-13-00-04 #PWR?
 U 1 1 5E9CE529
 P 6625 1600
@@
 	6850 2975 7150 2975
 $Comp
-L Envelope-cache-2018-08-04-13-00-04:GND #PWR?
+L KicadJE_Util-rescue:GND-Envelope-cache-2018-08-04-13-00-04 #PWR?
 U 1 1 5ECCE0BF
 P 7150 3700
@@
 $EndComp
 $Comp
-L Envelope-cache-2018-08-04-13-00-04:GND #PWR?
+L KicadJE_Util-rescue:GND-Envelope-cache-2018-08-04-13-00-04 #PWR?
 U 1 1 5ED09A0C
 P 7650 2075
